Commit message: added iur gripper finger stl and fixed xacro

File: wsg50_description/urdf/iiwa7_wsg50.xacro (robot description, xacro)
@@ -7,9 +7,4 @@
     <xacro:include filename="$(find lbr_description)/urdf/iiwa7/iiwa7_description.xacro" />
     <xacro:include filename="$(find wsg50_description)/urdf/wsg50.urdf.xacro" />
-    <link name="world" />
-    <joint name="$(arg robot_name)_world_joint" type="fixed">
-        <parent link="world" />
-        <child link="$(arg robot_name)_link_0" />
-    </joint>
     <xacro:iiwa7
         robot_name="$(arg robot_name)"
@@ -18,8 +13,6 @@
         initial_joint_positions_path="$(arg initial_joint_positions_path)" />
     <!-- Mechanical mounting of the WSG50 to the iiwa end-effector. -->
-    <xacro:wsg50 prefix="wsg50" parent="$(arg robot_name)_link_ee"
-                 finger_length="0.023" finger_tip="-0.001">
-        <!-- 50 degrees around the iiwa end-effector Z axis. -->
-        <origin xyz="0 0 0" rpy="0 0 0.872665" />
+    <xacro:wsg50 prefix="wsg50" parent="$(arg robot_name)_link_ee">
+        <origin xyz="0 0 0.011" rpy="0 0 0.8730137" />
     </xacro:wsg50>
 </robot>

File: wsg50_description/urdf/wsg50.urdf.xacro (robot description, xacro)
@@ -1,138 +1,18 @@
 <?xml version="1.0"?>
+<!-- WSG50-110 description adapted from KITrobotics/weiss_wsg50. -->
 <robot xmlns:xacro="http://www.ros.org/wiki/xacro">
-    <xacro:macro name="wsg50" params="prefix parent finger_length finger_tip *origin">
-        <joint name="${prefix}_gripper_joint" type="fixed">
-            <xacro:insert_block name="origin" />
-            <parent link="${parent}"/>
-            <child link="${prefix}_base_link"/>
-        </joint>
-         <link name="${prefix}_base_link">
-            <inertial>
-                <mass value="0.25" />
-                <origin xyz="0 0 0" />
-                <inertia  ixx="1.0" ixy="0.0"  ixz="0.0"  iyy="1.0"  iyz="0.0"  izz="1.0" />
-            </inertial>
-            <visual>
-                <origin xyz="0.0 0 0" rpy="0 0 0" />
-                <geometry>
-                    <box size="0.20 0.09 0.0735"/>
-                    <!-- <mesh filename="package://wsg50_description/meshes/WSG50_110.stl" scale="1 1 1"/> -->
-                </geometry>
-                <material name="grey">
-                <color rgba="0.5 0.5 0.5 1"/>
-                </material>
-            </visual>
-            <collision>
-                <origin xyz="0.0 0 0" rpy="0 0 0" />
-                <geometry>
-                    <box size="0.25 0.09 0.0735"/>
-                    <!-- <mesh filename="package://wsg50_description/meshes/WSG50_110.stl" scale="1 1 1"/> -->
-                </geometry>
-            </collision>
-        </link>
-        <gazebo reference="${prefix}_base_link">
-            <material>Gazebo/Grey</material>
-            <turnGravityOff>false</turnGravityOff>
-        </gazebo>
-        <joint name="${prefix}_center_joint" type="fixed">
-            <origin xyz="0 0 ${finger_length}" rpy="0 0 0" />      <!--origin xyz="-0.0067 0 0.049" rpy="0 0 0" /-->
-            <parent link="${prefix}_base_link"/>
-            <child link="${prefix}_center" />
-        </joint>
-        <link name="${prefix}_center" />
-        <!-- GRIPPER LEFT -->
-        <link name="${prefix}_gripper_left">
-            <inertial>
-                <mass value="0.1" />
-                <origin xyz="0 0 0" />
-                <inertia ixx="1.0" ixy="0.0" ixz="0.0"
-                    iyy="1.0" iyz="0.0"
-                    izz="1.0" />
-            </inertial>
-            <visual>
-                <origin xyz="0 0 0" rpy="0 0 0" />
-                <material name="grey" />
-                <geometry>
-                    <mesh filename="package://wsg50_description/meshes/kuka_gripper_2.dae" />
-                </geometry>
-            </visual>
-            <collision>
-                <origin xyz="0 0 0" rpy="0 0 0" />
-                <geometry>
-                    <mesh filename="package://wsg50_description/meshes/kuka_gripper_2.stl" />
-                </geometry>
-            </collision>
-            <contact_coefficients kd="1.0" kp="1000.0" mu="0"/>
-        </link>
-        <gazebo reference="${prefix}_gripper_left">
-            <material>Gazebo/Blue</material>
-            <turnGravityOff>false</turnGravityOff>
-        </gazebo>
-        <joint name="${prefix}_finger_left_joint" type="prismatic">
-            <origin xyz="0.08 0 0.12" rpy="3.1457 0 3.1457" />      <!--origin xyz="-0.0067 0 0.049" rpy="0 0 0" /-->
-            <parent link="${prefix}_base_link"/>
-            <child link="${prefix}_gripper_left" />
-            <dynamics friction="100" damping="100" />
-            <axis xyz="1 0 0"/>
-            <limit lower="-0.055" upper="0.0" effort="80.0" velocity="0.42"/>
-        </joint>
-         <!-- GRIPPER RIGHT -->
-        <link name="${prefix}_gripper_right">
-            <inertial>
-                <mass value="0.1" />
-                <origin xyz="0 0 0" />
-            <inertia ixx="1.0" ixy="0.0" ixz="0.0"
-                    iyy="1.0" iyz="0.0"
-                    izz="1.0" />
-            </inertial>
-            <visual>
-                <origin xyz="0.0 0 0" rpy="0 0 0" />
-                <material name="grey" />
-                <geometry>
-                    <mesh filename="package://wsg50_description/meshes/kuka_gripper_2.dae" />
-                </geometry>
-            </visual>
-            <collision>
-                <origin xyz="0 0 0" rpy="0 0 0" />
-                <geometry>
-                    <mesh filename="package://wsg50_description/meshes/kuka_gripper_2.stl"/>
-                </geometry>
-            </collision>
-            <contact_coefficients kd="1.0" kp="1000.0" mu="0"/>
-        </link>
-        <gazebo reference="${prefix}_gripper_right">
-            <material>Gazebo/White</material>
-            <turnGravityOff>false</turnGravityOff>
-        </gazebo>
-        <joint name="${prefix}_finger_right_joint" type="prismatic">
-            <origin xyz="-0.08 0 0.12" rpy="3.14159 0 0" />
-            <parent link="${prefix}_base_link"/>
-            <child link="${prefix}_gripper_right" />
-            <axis xyz="-1 0 0"/>
-            <dynamics friction="100" damping="100" />
-            <limit lower="0.0" upper="0.055" effort="80.0" velocity="0.42"/>
-        </joint>
-        <!-- <link name="object">
-            <inertial>
-                <mass value="100"/>
-                <origin xyz="0 0 0" />
-                <inertia  ixx="1" ixy="0.0"  ixz="0.0"  iyy="1"  iyz="0.0"  izz="1" />
-            </inertial>
-            <visual>
-                <origin rpy="0 0 0" xyz="0 0 0"/>
-                <geometry>
-                    <box size="0.08 0.08 0.4"/>
-                </geometry>
-                <material name="white">
-                    <color rgba="1.0 1.0 1.0 1.0"/>
-                </material>
-            </visual>
-            <collision>
-                <origin rpy="0 0 0" xyz="0 0 0"/>
-                <geometry>
-                    <box size="0.08 0.08 0.4"/>
-                </geometry>
-            </collision>
-        </link> -->
-    </xacro:macro>
+  <material name="wsg50_gray"><color rgba="0.45 0.45 0.45 1.0"/></material>
+  <material name="wsg50_dark_green"><color rgba="0.02 0.22 0.06 1.0"/></material>
+  <xacro:macro name="wsg50" params="prefix parent *origin">
+    <joint name="${prefix}_palm_joint" type="fixed"><xacro:insert_block name="origin"/><parent link="${parent}"/><child link="${prefix}_palm_link"/></joint>
+    <link name="${prefix}_palm_link">
+      <inertial><mass value="0.25"/><origin xyz="0 0 0"/><inertia ixx="1.0" ixy="0" ixz="0" iyy="1.0" iyz="0" izz="1.0"/></inertial>
+      <visual><geometry><mesh filename="package://wsg50_description/meshes/WSG50_110.stl"/></geometry><material name="wsg50_gray"/></visual>
+      <collision><geometry><mesh filename="package://wsg50_description/meshes/WSG50_110.stl" scale="0.001 0.001 0.001"/></geometry></collision>
+    </link>
+    <joint name="${prefix}_finger_left_joint" type="prismatic"><origin xyz="0 0 0.0819"/><parent link="${prefix}_palm_link"/><child link="${prefix}_finger_left_link"/><axis xyz="-1 0 0"/><limit effort="10" lower="-0.055" upper="0" velocity="0.42"/></joint>
+    <link name="${prefix}_finger_left_link"><inertial><mass value="0.25"/><origin xyz="0 0 0"/><inertia ixx="1.0" ixy="0" ixz="0" iyy="1.0" iyz="0" izz="1.0"/></inertial><visual><origin xyz="0.01975 0 0" rpy="1.5707963267948966 3.141592653589793 -1.5707963267948966"/><geometry><mesh filename="package://wsg50_description/meshes/Kuka_Greifer.STL" scale="0.001 0.001 0.001"/></geometry><material name="wsg50_dark_green"/></visual><collision><origin xyz="0.01975 0 0" rpy="1.5707963267948966 3.141592653589793 -1.5707963267948966"/><geometry><mesh filename="package://wsg50_description/meshes/Kuka_Greifer.STL" scale="0.001 0.001 0.001"/></geometry></collision></link>
+    <joint name="${prefix}_finger_right_joint" type="prismatic"><origin xyz="0 0 0.0819" rpy="0 0 ${pi}"/><parent link="${prefix}_palm_link"/><child link="${prefix}_finger_right_link"/><axis xyz="1 0 0"/><limit effort="10" lower="0" upper="0.055" velocity="0.42"/></joint>
+    <link name="${prefix}_finger_right_link"><inertial><mass value="0.25"/><origin xyz="0 0 0"/><inertia ixx="1.0" ixy="0" ixz="0" iyy="1.0" iyz="0" izz="1.0"/></inertial><visual><origin xyz="0.0235 0 0" rpy="1.5707963267948966 3.141592653589793 -1.5707963267948966"/><geometry><mesh filename="package://wsg50_description/meshes/Kuka_Greifer.STL" scale="0.001 0.001 0.001"/></geometry><material name="wsg50_dark_green"/></visual><collision><origin xyz="0.0235 0 0" rpy="1.5707963267948966 3.141592653589793 -1.5707963267948966"/><geometry><mesh filename="package://wsg50_description/meshes/Kuka_Greifer.STL" scale="0.001 0.001 0.001"/></geometry></collision></link>
+  </xacro:macro>
 </robot>

File: wsg50_description/urdf/wsg50.xacro (robot description, xacro)
@@ -11,5 +11,5 @@
     </gazebo>
     <!-- World to table -->
-    <xacro:wsg50 prefix="wsg50" parent="world" finger_length="0.023" finger_tip="-0.001">
+    <xacro:wsg50 prefix="wsg50" parent="world">
         <origin xyz="0 0 1" rpy="0 0 0" />
     </xacro:wsg50>
